File: Templates/CubeSatKit_StackBoard/CubeSatKit_StackBoard.kicad_pcb (KiCad board)
At the start: 2 copper layers, 90.2 x 95.9 mm, 6 parts

Commit message: Updated CubeSat template
Parts:
- H1, H2: footprint CSK_Header -> Connectors:CONN_2.54mm_2x26
Connections:
- H1 pad 1: (no net) -> Net-(H1-Pad1)
- H1 pad 10: (no net) -> Net-(H1-Pad10)
- H1 pad 11: (no net) -> Net-(H1-Pad11)
- H1 pad 12: (no net) -> Net-(H1-Pad12)
- H1 pad 13: (no net) -> Net-(H1-Pad13)
- H1 pad 14: (no net) -> Net-(H1-Pad14)
- H1 pad 15: (no net) -> Net-(H1-Pad15)
- H1 pad 16: (no net) -> Net-(H1-Pad16)
- H1 pad 17: (no net) -> Net-(H1-Pad17)
- H1 pad 18: (no net) -> Net-(H1-Pad18)
- H1 pad 19: (no net) -> Net-(H1-Pad19)
- H1 pad 2: (no net) -> Net-(H1-Pad2)
- H1 pad 20: (no net) -> Net-(H1-Pad20)
- H1 pad 21: (no net) -> Net-(H1-Pad21)
- H1 pad 22: (no net) -> Net-(H1-Pad22)
- H1 pad 23: (no net) -> Net-(H1-Pad23)
- H1 pad 24: (no net) -> Net-(H1-Pad24)
- H1 pad 25: (no net) -> Net-(H1-Pad25)
- H1 pad 26: (no net) -> Net-(H1-Pad26)
- H1 pad 27: (no net) -> Net-(H1-Pad27)
- H1 pad 28: (no net) -> Net-(H1-Pad28)
- H1 pad 29: (no net) -> Net-(H1-Pad29)
- H1 pad 3: (no net) -> Net-(H1-Pad3)
- H1 pad 30: (no net) -> Net-(H1-Pad30)
- H1 pad 31: (no net) -> Net-(H1-Pad31)
- H1 pad 32: (no net) -> Net-(H1-Pad32)
- H1 pad 33: (no net) -> Net-(H1-Pad33)
- H1 pad 34: (no net) -> Net-(H1-Pad34)
- H1 pad 35: (no net) -> Net-(H1-Pad35)
- H1 pad 36: (no net) -> Net-(H1-Pad36)
- H1 pad 37: (no net) -> Net-(H1-Pad37)
- H1 pad 38: (no net) -> Net-(H1-Pad38)
- H1 pad 39: (no net) -> Net-(H1-Pad39)
- H1 pad 4: (no net) -> Net-(H1-Pad4)
- H1 pad 40: (no net) -> Net-(H1-Pad40)
- H1 pad 41: (no net) -> Net-(H1-Pad41)
- H1 pad 42: (no net) -> Net-(H1-Pad42)
- H1 pad 43: (no net) -> Net-(H1-Pad43)
- H1 pad 44: (no net) -> Net-(H1-Pad44)
- H1 pad 45: (no net) -> Net-(H1-Pad45)
- H1 pad 46: (no net) -> Net-(H1-Pad46)
- H1 pad 47: (no net) -> Net-(H1-Pad47)
- H1 pad 48: (no net) -> Net-(H1-Pad48)
- H1 pad 49: (no net) -> Net-(H1-Pad49)
- H1 pad 5: (no net) -> Net-(H1-Pad5)
- H1 pad 50: (no net) -> Net-(H1-Pad50)
- H1 pad 51: (no net) -> Net-(H1-Pad51)
- H1 pad 52: (no net) -> Net-(H1-Pad52)
- H1 pad 6: (no net) -> Net-(H1-Pad6)
- H1 pad 7: (no net) -> Net-(H1-Pad7)
- H1 pad 8: (no net) -> Net-(H1-Pad8)
- H1 pad 9: (no net) -> Net-(H1-Pad9)
- H2 pad 1: (no net) -> Net-(H2-Pad1)
- H2 pad 10: (no net) -> Net-(H2-Pad10)
- H2 pad 11: (no net) -> Net-(H2-Pad11)
- H2 pad 12: (no net) -> Net-(H2-Pad12)
- H2 pad 13: (no net) -> Net-(H2-Pad13)
- H2 pad 14: (no net) -> Net-(H2-Pad14)
- H2 pad 15: (no net) -> Net-(H2-Pad15)
- H2 pad 16: (no net) -> Net-(H2-Pad16)
- H2 pad 17: (no net) -> Net-(H2-Pad17)
- H2 pad 18: (no net) -> Net-(H2-Pad18)
- H2 pad 19: (no net) -> Net-(H2-Pad19)
- H2 pad 2: (no net) -> Net-(H2-Pad2)
- H2 pad 20: (no net) -> Net-(H2-Pad20)
- H2 pad 21: (no net) -> Net-(H2-Pad21)
- H2 pad 22: (no net) -> Net-(H2-Pad22)
- H2 pad 23: (no net) -> Net-(H2-Pad23)
- H2 pad 24: (no net) -> Net-(H2-Pad24)
- H2 pad 25: (no net) -> Net-(H2-Pad25)
- H2 pad 26: (no net) -> Net-(H2-Pad26)
- H2 pad 27: (no net) -> Net-(H2-Pad27)
- H2 pad 28: (no net) -> Net-(H2-Pad28)
- H2 pad 29: (no net) -> Net-(H2-Pad29)
- H2 pad 3: (no net) -> Net-(H2-Pad3)
- H2 pad 30: (no net) -> Net-(H2-Pad30)
- H2 pad 31: (no net) -> Net-(H2-Pad31)
- H2 pad 32: (no net) -> Net-(H2-Pad32)
- H2 pad 33: (no net) -> Net-(H2-Pad33)
- H2 pad 34: (no net) -> Net-(H2-Pad34)
- H2 pad 35: (no net) -> Net-(H2-Pad35)
- H2 pad 36: (no net) -> Net-(H2-Pad36)
- H2 pad 37: (no net) -> Net-(H2-Pad37)
- H2 pad 38: (no net) -> Net-(H2-Pad38)
- H2 pad 39: (no net) -> Net-(H2-Pad39)
- H2 pad 4: (no net) -> Net-(H2-Pad4)
- H2 pad 40: (no net) -> Net-(H2-Pad40)
- H2 pad 41: (no net) -> Net-(H2-Pad41)
- H2 pad 42: (no net) -> Net-(H2-Pad42)
- H2 pad 43: (no net) -> Net-(H2-Pad43)
- H2 pad 44: (no net) -> Net-(H2-Pad44)
- H2 pad 45: (no net) -> Net-(H2-Pad45)
- H2 pad 46: (no net) -> Net-(H2-Pad46)
- H2 pad 47: (no net) -> Net-(H2-Pad47)
- H2 pad 48: (no net) -> Net-(H2-Pad48)
- H2 pad 49: (no net) -> Net-(H2-Pad49)
- H2 pad 5: (no net) -> Net-(H2-Pad5)
- H2 pad 50: (no net) -> Net-(H2-Pad50)
- H2 pad 51: (no net) -> Net-(H2-Pad51)
- H2 pad 52: (no net) -> Net-(H2-Pad52)
- H2 pad 6: (no net) -> Net-(H2-Pad6)
- H2 pad 7: (no net) -> Net-(H2-Pad7)
- H2 pad 8: (no net) -> Net-(H2-Pad8)
- H2 pad 9: (no net) -> Net-(H2-Pad9)
