File: Templates/CubeSatKit_StackBoard/CubeSatKit_StackBoard.sch (KiCad schematic (older format))
At the start: 2 parts

Commit message: Updated CubeSat template
Parts:
- H1, H2: footprint (none) -> Connectors:CONN_2.54mm_2x26
Changed lines of the file:
@@
 LIBS:memory
 LIBS:xilinx
-LIBS:special
 LIBS:microcontrollers
 LIBS:dsp
@@
 LIBS:contrib
 LIBS:valves
-LIBS:MiscellaneousDevices
 LIBS:CubeSatKit_StackBoard-cache
-EELAYER 27 0
+EELAYER 25 0
 EELAYER END
 $Descr A4 11693 8268
@@
 F 0 "H2" H 9800 3850 60  0000 C CNN
 F 1 "H2" V 9800 2450 60  0000 C CNN
-F 2 "" H 9800 2500 60  0001 C CNN
+F 2 "Connectors:CONN_2.54mm_2x26" H 9800 2500 60  0001 C CNN
 F 3 "" H 9800 2500 60  0001 C CNN
 	1    9800 2500
@@
 F 0 "H1" H 8400 3850 60  0000 C CNN
 F 1 "H1" V 8400 2450 60  0000 C CNN
-F 2 "" H 8400 2500 60  0001 C CNN
+F 2 "Connectors:CONN_2.54mm_2x26" H 8400 2500 60  0001 C CNN
 F 3 "" H 8400 2500 60  0001 C CNN
 	1    8400 2500
